File: Extensions/Buttons/Button PCB.kicad_pcb (KiCad board)
At the start: 2 copper layers, 29.9 x 14.5 mm, 7 parts, among them P1 Solder_Pad, P2 Solder_Pad, P3 Solder_Pad, SW1 TS-1102S-C-A-B, SW2 TS-1102S-C-A-B

Commit message: added second schottky diode for less heat
Parts:
- removed qrcode: LOGO, LOGO
- added G***: LOGO, LOGO, B.Cu at (131.0, 99.4)
Other:
- board text added: "PCB files: https://bit.ly/ 3Idt9md"
- board text removed: "PCB files: https://bit.ly/ ...."
