File: Extensions/Buttons/Button PCB.kicad_sch (KiCad schematic)
At the start: 5 parts, among them P2 Solder_Pad, P3 Solder_Pad, SW1 TS-1102S-C-A-B, SW2 TS-1102S-C-A-B

Commit message: added second schottky diode for less heat
Parts:
- P1: now left out of the parts list
- P2, P3: value Solder_Pad -> (none); footprint footprint:Solder pad -> (none); now left out of the parts list
Changed lines of the file:
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@@
   )
   (symbol (lib_id "MyParts:Solder_Pad") (at 129.54 68.58 0) (unit 1)
-    (in_bom yes) (on_board yes) (fields_autoplaced)
+    (in_bom no) (on_board yes) (fields_autoplaced)
     (property "Reference" "P2" (id 0) (at 138.43 67.3099 0)
       (effects (font (size 1.27 1.27)) (justify left))
     )
-    (property "Value" "Solder_Pad" (id 1) (at 138.43 69.8499 0)
+    (property "Value" "" (id 1) (at 138.43 69.8499 0)
       (effects (font (size 1.27 1.27)) (justify left))
     )
-    (property "Footprint" "footprint:Solder pad" (id 2) (at 129.54 68.58 0)
+    (property "Footprint" "" (id 2) (at 129.54 68.58 0)
       (effects (font (size 1.27 1.27)) hide)
     )
@@
   )
   (symbol (lib_id "MyParts:Solder_Pad") (at 129.54 74.93 0) (unit 1)
-    (in_bom yes) (on_board yes) (fields_autoplaced)
+    (in_bom no) (on_board yes) (fields_autoplaced)
     (property "Reference" "P3" (id 0) (at 138.43 73.6599 0)
       (effects (font (size 1.27 1.27)) (justify left))
     )
-    (property "Value" "Solder_Pad" (id 1) (at 138.43 76.1999 0)
+    (property "Value" "" (id 1) (at 138.43 76.1999 0)
       (effects (font (size 1.27 1.27)) (justify left))
     )
-    (property "Footprint" "footprint:Solder pad" (id 2) (at 129.54 74.93 0)
+    (property "Footprint" "" (id 2) (at 129.54 74.93 0)
       (effects (font (size 1.27 1.27)) hide)
     )
@@
   )
   (symbol (lib_id "MyParts:Solder_Pad") (at 129.54 62.23 0) (unit 1)
-    (in_bom yes) (on_board yes) (fields_autoplaced)
+    (in_bom no) (on_board yes) (fields_autoplaced)
     (property "Reference" "P1" (id 0) (at 138.43 60.9599 0)
       (effects (font (size 1.27 1.27)) (justify left))
