File: GlowCore PCB/GlowCore.kicad_pcb (KiCad board)
At the start: 4 copper layers, 20 x 38 mm, 59 parts, among them P1 Solder_Pad, P10 Solder_Pad, P11 Solder_Pad, P12 Solder_Pad, P13 Solder_Pad, P14 Solder_Pad, P15 Solder_Pad, P16 Solder_Pad, P17 Solder_Pad, P18 Solder_Pad, P19 Solder_Pad, P2 Solder_Pad, P20 Solder_Pad, P21 Solder_Pad, P22 Solder_Pad, P23 Solder_Pad, P24 Solder_Pad, P3 Solder_Pad, P4 Solder_Pad, P5 Solder_Pad, P6 Solder_Pad, P7 Solder_Pad, P8 Solder_Pad, P9 Solder_Pad, SW1 TS24CA, SW2 TS24CA, SW3 TS24CA, U1 SN74LVC1G373DBVR, U10 AP40P05, U11 74LVC2G04DW-7, U2 AP40P05, U3 ESP32-S3-MINI-1-N8, U4 AP40P05, U5 AO3400A, U6 SN74LVC2T45DCUR, U7 SPX3819M5-L-3-3_TR, U8 SK9822-EC20, U9 AP40P05

Commit message: update folder structure
Parts:
- moved P12 0.06 mm to (163.0, 71.2)
- moved P13 0.06 mm to (165.9, 71.2)
- moved P23 0.06 mm to (160.1, 71.2)
- moved P24 0.06 mm to (157.2, 71.2)
- moved P7 0.06 mm to (151.4, 71.2)
- moved P8 0.06 mm to (154.3, 71.2)
Routing:
- net GND: track 130.0 -> 128.9 mm, vias 103 -> 100
- net Net-(U10-G): track 19.9 -> 18.9 mm
- net 3.3V AFTER MOSFET: track 10.0 -> 9.05 mm
