File: GlowCore PCB/GlowCore.kicad_sch (KiCad schematic)
At the start: 59 parts, among them P1 Solder_Pad, P10 Solder_Pad, P11 Solder_Pad, P12 Solder_Pad, P13 Solder_Pad, P14 Solder_Pad, P15 Solder_Pad, P16 Solder_Pad, P17 Solder_Pad, P18 Solder_Pad, P19 Solder_Pad, P2 Solder_Pad, P20 Solder_Pad, P21 Solder_Pad, P22 Solder_Pad, P23 Solder_Pad, P24 Solder_Pad, P3 Solder_Pad, P4 Solder_Pad, P5 Solder_Pad, P6 Solder_Pad, P7 Solder_Pad, P8 Solder_Pad, P9 Solder_Pad, SW1 TS24CA, SW2 TS24CA, SW3 TS24CA, U1 SN74LVC1G373DBVR, U10 AP40P05, U11 74LVC2G04DW-7, U2 AP40P05, U3 ESP32-S3-MINI-1-N8, U4 AP40P05, U5 AO3400A, U6 SN74LVC2T45DCUR, U7 SPX3819M5-L-3-3_TR, U8 SK9822-EC20, U9 AP40P05

Commit message: update folder structure
Other:
- moved on the sheet: C1, C2, C3, C4, C5, C6, C7, C8, P1, P10, P11, P12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

Commit message: updated pcb design
Parts:
- removed R13, R14, R3, R4, R5: 100K, Resistor_SMD:R_0402_1005Metric, symbol Device:10K 0603
- removed U1: SN74LVC1G373DBVR, footprint:SOT-23-6_L2.9-W1.6-P0.95-LS2.8-BR, symbol MyParts:SN74LVC1G373DBVR
- removed U10, U2, U4, U9: AP40P05, footprint:SOT-23-3_L2.9-W1.3-P1.90-LS2.4-BR, symbol MyParts:AP40P05
- removed U5: AO3400A, footprint:SOT-23-3_L2.9-W1.6-P1.90-LS2.8-BR, symbol MyParts:AO3400A
- removed U8: SK9822-EC20, footprint:LED-SMD_6P-L2.0-W2.0-P0.80-TL, symbol MyParts:SK9822-EC20
- added U1: SK9822-EC20, footprint:LED-SMD_6P-L2.0-W2.0-P0.80-TL, symbol MyParts:SK9822-EC20
- U3: value ESP32-S3-MINI-1-N8 -> ESP32-S3-MINI-1-N4R2; LCSC# C2913206 -> C3013941
Connections:
- net 3.3V AFTER MOSFET is gone; now on net +3V3: C5.1, P18.1, U6.8 (VCCB)
- net 5V AFTER MOSFET is gone; now on net VBUS: C4.1, P1.1, P4.1, U6.1 (VCCA)
- net GND: now also SW1.1, SW1.2, SW2.1, SW2.2, SW3.1, SW3.2, U1.2 (GND)
- net IO39/STATUS LED CLOCK: now also U1.4 (CKL)
- net IO40/STATUS LED DATA: now also U1.3 (SDI)
- net VBUS: now also U1.5 (VDD)
- net IO15/LED LETCH EN: no longer names the net of U3.19 (IO15)
- net IO16/POWERMOSFETS: no longer names the net of U3.20 (IO16)
- no-connect marks 29 -> 24
Other:
- note added: "Levelshifter + LED pads"
- note removed: "LED power"
- note removed: "LED strip pads"
- moved on the sheet: C3, C4, C5, C6, C7, C8, P1, P2, P3, P4, P5, P6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
